File: Simple/Simple.sch (EAGLE design)
At the start: 30 parts, among them IC1 LM7805, IC2 AVR-MEGA8-PPTH, IC3 MCP1700-33, J1 ISP, J4 VIN, Y1 16MHz

Commit message: Added IOREF and reserved pins
Parts:
- POWER: value (none) -> POWER; device SparkFun:M06SIP -> SparkFun:M081X08
Connections:
- new net RESERVED: POWER.1
- net 3.3V: now also POWER.4; no longer POWER.2
- net 5V: now also POWER.5; no longer POWER.3
- net GND: now also POWER.6, POWER.7; no longer POWER.4, POWER.5
- net RESET: now also POWER.3; no longer POWER.1
- net VIN: now also POWER.8; no longer POWER.6
Changed lines of the file:
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@@
 <part name="GND1" library="SparkFun" deviceset="GND" device=""/>
 <part name="C1" library="SparkFun" deviceset="CAP" device="PTH2" value="0.1uF"/>
-<part name="POWER" library="SparkFun" deviceset="M06" device="SIP"/>
 <part name="R1" library="SparkFun" deviceset="RESISTOR" device="AXIAL-0.3" value="330"/>
 <part name="LED1" library="SparkFun" deviceset="LED" device="5MM" value="RED"/>
@@
 <part name="IOH" library="SparkFun-Connectors" deviceset="CONN_10" device="&quot;" value="IOH"/>
 <part name="FRAME2" library="SparkFun-Aesthetics" deviceset="FRAME-LETTER" device=""/>
+<part name="POWER" library="SparkFun" deviceset="M08" device="1X08" value="POWER"/>
 </parts>
 <sheets>
@@
 <attribute name="NAME" x="98.044" y="68.961" size="1.778" layer="95"/>
 <attribute name="VALUE" x="93.599" y="65.024" size="1.778" layer="96" rot="R90"/>
-</instance>
-<instance part="POWER" gate="G$1" x="175.26" y="119.38" smashed="yes" rot="R180">
-<attribute name="NAME" x="179.578" y="114.3" size="1.778" layer="95" rot="R90"/>
-<attribute name="VALUE" x="180.34" y="129.54" size="1.778" layer="96" rot="R180"/>
 </instance>
 <instance part="R1" gate="G$1" x="149.86" y="43.18" rot="R180"/>
@@
 <instance part="FRAME2" gate="G$1" x="0" y="0"/>
 <instance part="FRAME2" gate="V" x="147.32" y="0"/>
+<instance part="POWER" gate="G$1" x="175.26" y="121.92" smashed="yes" rot="R180">
+<attribute name="NAME" x="179.578" y="119.126" size="1.778" layer="95" rot="R90"/>
+</instance>
 </instances>
 <busses>
@@
 <wire x1="160.02" y1="119.38" x2="170.18" y2="119.38" width="0.1524" layer="91"/>
 <label x="160.02" y="119.38" size="1.778" layer="95"/>
-<pinref part="POWER" gate="G$1" pin="3"/>
+<pinref part="POWER" gate="G$1" pin="5"/>
 </segment>
 <segment>
@@
 <pinref part="R2" gate="G$1" pin="2"/>
 </segment>
+<segment>
+<wire x1="160.02" y1="127" x2="170.18" y2="127" width="0.1524" layer="91"/>
+<label x="160.02" y="127" size="1.778" layer="95"/>
+</segment>
 </net>
 <net name="GND" class="0">
@@
 <wire x1="170.18" y1="116.84" x2="160.02" y2="116.84" width="0.1524" layer="91"/>
 <label x="160.02" y="116.84" size="1.778" layer="95"/>
-<pinref part="POWER" gate="G$1" pin="4"/>
+<pinref part="POWER" gate="G$1" pin="6"/>
 </segment>
 <segment>
 <wire x1="170.18" y1="114.3" x2="160.02" y2="114.3" width="0.1524" layer="91"/>
 <label x="160.02" y="114.3" size="1.778" layer="95"/>
-<pinref part="POWER" gate="G$1" pin="5"/>
+<pinref part="POWER" gate="G$1" pin="7"/>
 </segment>
 <segment>
@@
 <wire x1="170.18" y1="124.46" x2="160.02" y2="124.46" width="0.1524" layer="91"/>
 <label x="160.02" y="124.46" size="1.778" layer="95"/>
-<pinref part="POWER" gate="G$1" pin="1"/>
+<pinref part="POWER" gate="G$1" pin="3"/>
 </segment>
 <segment>
@@
 <wire x1="170.18" y1="121.92" x2="160.02" y2="121.92" width="0.1524" layer="91"/>
 <label x="160.02" y="121.92" size="1.778" layer="95"/>
-<pinref part="POWER" gate="G$1" pin="2"/>
+<pinref part="POWER" gate="G$1" pin="4"/>
 </segment>
 <segment>
@@
 <wire x1="160.02" y1="111.76" x2="170.18" y2="111.76" width="0.1524" layer="91"/>
 <label x="160.02" y="111.76" size="1.778" layer="95"/>
-<pinref part="POWER" gate="G$1" pin="6"/>
+<pinref part="POWER" gate="G$1" pin="8"/>
 </segment>
 <segment>
@@
 </segment>
 </net>
+<net name="RESERVED" class="0">
+<segment>
+<pinref part="POWER" gate="G$1" pin="1"/>
+<wire x1="170.18" y1="129.54" x2="160.02" y2="129.54" width="0.1524" layer="91"/>
+<label x="160.02" y="129.54" size="1.778" layer="95"/>
+</segment>
+</net>
